File: BrainPower/BrainPower.kicad_pcb (KiCad board)
At the start: 2 copper layers, 150 x 111.3 mm, 10 parts, among them J1 BarrelJack_Horizontal, J2 PhoenixContact_MCV_1,5_2-G-5.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, P1 Golden finger, PCIeX1, Dual, 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

Commit message: add some silkscreen words
Other:
- board text added: "[Emergency Only] Cut the trace to activate the firewall!"
- board text added: "^"
Changed lines of the file:
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@@
   (general
     (thickness 1.6)
-    (drawings 43)
+    (drawings 48)
     (tracks 47)
     (zones 0)
@@
     (pad A17 smd rect (at 8.5 0) (size 0.7 4.2) (layers B.Cu B.Paste B.Mask))
   )
+  (gr_arc (start 175.6 130.8) (end 180.3 128.1) (angle -55.88761251) (layer F.SilkS) (width 0.15))
+  (gr_circle (center 180.9 130.9) (end 182.5 132.5) (layer F.SilkS) (width 0.15))
+  (gr_text ^ (at 180.9 132.8) (layer F.SilkS)
+    (effects (font (size 1.5 1.5) (thickness 0.2)))
+  )
+  (gr_text ^ (at 180.9 129.1 180) (layer F.SilkS)
+    (effects (font (size 1.5 1.5) (thickness 0.2)))
+  )
+  (gr_text "[Emergency Only]\nCut the trace to activate the firewall!" (at 117.5 123.8) (layer F.SilkS)
+    (effects (font (size 2 2) (thickness 0.25)) (justify left))
+  )
   (gr_text "BrainPower Version 0.2\nhttps://github.com/Jamesits/BrainPower" (at 83 67 90) (layer B.SilkS)

Commit message: add compatibility with low profile PCI express I/O brackets
Parts:
- added MH2: MountingHole_3.2mm_M3_ISO14580_Pad, MountingHole:MountingHole_3.2mm_M3_ISO14580_Pad, F.Cu at (80.8, 92.6)
- moved MH1 0.26 mm to (80.8, 146.5)
- renumbered MH2 to MH3
Other:
- board text added: "0.3"
- board text added: "2019-11-07"
- board text added: "BrainPower Version 0.3 https://github.com/Jamesits/BrainPower"
- board text added: "Note: Tolerance ±0.13"
- board text removed: "0.2"
- board text removed: "2019-10-16"
- board text removed: "BrainPower Version 0.2 https://github.com/Jamesits/BrainPower"
Changed lines of the file:
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@@
   (general
     (thickness 1.6)
-    (drawings 48)
+    (drawings 54)
     (tracks 47)
     (zones 0)
-    (modules 10)
+    (modules 11)
     (nets 3)
   )
@@
     (pad_to_mask_clearance 0)
     (aux_axis_origin 0 0)
+    (grid_origin 73.33 151.3796)
     (visible_elements 7FFFFF7F)
     (pcbplotparams
@@
     (diff_pair_width 0.254)
     (diff_pair_gap 0.25)
+  )
+  (module MountingHole:MountingHole_3.2mm_M3_ISO14580_Pad (layer F.Cu)
+    (at 80.83 92.63)
+    (descr "Mounting Hole 3.2mm, M3, ISO14580")
+    (tags "mounting hole 3.2mm m3 iso14580")
+    (attr virtual)
+    (fp_text reference MH2 (at 0 -3.75) (layer F.SilkS) hide
+      (effects (font (size 1 1) (thickness 0.15)))
+    )
+    (fp_text value MountingHole_3.2mm_M3_ISO14580_Pad (at 0 3.75) (layer F.Fab)
+      (effects (font (size 1 1) (thickness 0.15)))
+    )
+    (fp_text user %R (at 0.3 0) (layer F.Fab)
+      (effects (font (size 1 1) (thickness 0.15)))
+    )
+    (fp_circle (center 0 0) (end 2.75 0) (layer Cmts.User) (width 0.15))
+    (fp_circle (center 0 0) (end 3 0) (layer F.CrtYd) (width 0.05))
+    (pad 1 thru_hole circle (at 0 0) (size 5.5 5.5) (drill 3.2) (layers *.Cu *.Mask))
   )
   (module Footprints:RB750Gr3 (layer F.Cu)
@@
   )
   (module MountingHole:MountingHole_3.2mm_M3_ISO14580_Pad (layer F.Cu)
-    (at 80.8228 61.1378)
+    (at 80.83 61.13)
     (descr "Mounting Hole 3.2mm, M3, ISO14580")
     (tags "mounting hole 3.2mm m3 iso14580")
     (attr virtual)
-    (fp_text reference MH2 (at 0 -3.75) (layer F.SilkS)
+    (fp_text reference MH3 (at 0 -3.75) (layer F.SilkS) hide
       (effects (font (size 1 1) (thickness 0.15)))
     )
@@
   )
   (module MountingHole:MountingHole_3.2mm_M3_ISO14580_Pad (layer F.Cu)
-    (at 80.5688 146.5072)
+    (at 80.83 146.53)
     (descr "Mounting Hole 3.2mm, M3, ISO14580")
     (tags "mounting hole 3.2mm m3 iso14580")
     (attr virtual)
-    (fp_text reference MH1 (at 0 -3.75) (layer F.SilkS)
+    (fp_text reference MH1 (at 0 -3.75) (layer F.SilkS) hide
       (effects (font (size 1 1) (thickness 0.15)))
     )
@@
     (pad A17 smd rect (at 8.5 0) (size 0.7 4.2) (layers B.Cu B.Paste B.Mask))
   )
+  (dimension 84.700129 (width 0.15) (layer Dwgs.User)
+    (gr_text "84.700 mm" (at 181.007636 158.880392 0.1000611935) (layer Dwgs.User)
+      (effects (font (size 1 1) (thickness 0.15)))
+    )
+    (feature1 (pts (xy 223.33 142.98168) (xy 223.35639 158.092854)))
+    (feature2 (pts (xy 138.63 143.1296) (xy 138.65639 158.240774)))
+    (crossbar (pts (xy 138.655366 157.654354) (xy 223.355366 157.506434)))
+    (arrow1a (pts (xy 223.355366 157.506434) (xy 222.229888 158.094821)))
+    (arrow1b (pts (xy 223.355366 157.506434) (xy 222.22784 156.921981)))
+    (arrow2a (pts (xy 138.655366 157.654354) (xy 139.782892 158.238807)))
+    (arrow2b (pts (xy 138.655366 157.654354) (xy 139.780844 157.065967)))
+  )
+  (dimension 8 (width 0.15) (layer Dwgs.User)
+    (gr_text "8.000 mm" (at 110.68 158.9296) (layer Dwgs.User)
+      (effects (font (size 1 1) (thickness 0.15)))
+    )
+    (feature1 (pts (xy 114.68 151.3796) (xy 114.68 158.216021)))
+    (feature2 (pts (xy 106.68 151.3796) (xy 106.68 158.216021)))
+    (crossbar (pts (xy 106.68 157.6296) (xy 114.68 157.6296)))
+    (arrow1a (pts (xy 114.68 157.6296) (xy 113.553496 158.216021)))
+    (arrow1b (pts (xy 114.68 157.6296) (xy 113.553496 157.043179)))
+    (arrow2a (pts (xy 106.68 157.6296) (xy 107.806504 158.216021)))
+    (arrow2b (pts (xy 106.68 157.6296) (xy 107.806504 157.043179)))
+  )
+  (dimension 18.35 (width 0.15) (layer Dwgs.User)
+    (gr_text "18.350 mm" (at 97.505 158.929599) (layer Dwgs.User)
+      (effects (font (size 1 1) (thickness 0.15)))
+    )
+    (feature1 (pts (xy 106.68 151.3796) (xy 106.68 158.21602)))
+    (feature2 (pts (xy 88.33 151.3796) (xy 88.33 158.21602)))
+    (crossbar (pts (xy 88.33 157.629599) (xy 106.68 157.629599)))
+    (arrow1a (pts (xy 106.68 157.629599) (xy 105.553496 158.21602)))
+    (arrow1b (pts (xy 106.68 157.629599) (xy 105.553496 157.043178)))
+    (arrow2a (pts (xy 88.33 157.629599) (xy 89.456504 158.21602)))
+    (arrow2b (pts (xy 88.33 157.629599) (xy 89.456504 157.043178)))
+  )
+  (gr_text "Note:\nTolerance ±0.13" (at 178.38 168.0796) (layer Cmts.User)
+    (effects (font (size 1 1) (thickness 0.15)) (justify left))
+  )
+  (dimension 31.5 (width 0.15) (layer Dwgs.User)
+    (gr_text "31.500 mm" (at 62.03 76.88 90) (layer Dwgs.User)
+      (effects (font (size 1 1) (thickness 0.15)))
+    )
+    (feature1 (pts (xy 80.83 61.13) (xy 62.743579 61.13)))
+    (feature2 (pts (xy 80.83 92.63) (xy 62.743579 92.63)))
+    (crossbar (pts (xy 63.33 92.63) (xy 63.33 61.13)))
+    (arrow1a (pts (xy 63.33 61.13) (xy 63.916421 62.256504)))
+    (arrow1b (pts (xy 63.33 61.13) (xy 62.743579 62.256504)))
+    (arrow2a (pts (xy 63.33 92.63) (xy 63.916421 91.503496)))
+    (arrow2b (pts (xy 63.33 92.63) (xy 62.743579 91.503496)))
+  )
+  (dimension 53.9 (width 0.15) (layer Dwgs.User)
+    (gr_text "53.900 mm" (at 62.03 119.58 90) (layer Dwgs.User)
+      (effects (font (size 1 1) (thickness 0.15)))
+    )
+    (feature1 (pts (xy 80.83 92.63) (xy 62.743579 92.63)))
+    (feature2 (pts (xy 80.83 146.53) (xy 62.743579 146.53)))
+    (crossbar (pts (xy 63.33 146.53) (xy 63.33 92.63)))
+    (arrow1a (pts (xy 63.33 92.63) (xy 63.916421 93.756504)))
+    (arrow1b (pts (xy 63.33 92.63) (xy 62.743579 93.756504)))
+    (arrow2a (pts (xy 63.33 146.53) (xy 63.916421 145.403496)))
+    (arrow2b (pts (xy 63.33 146.53) (xy 62.743579 145.403496)))
+  )
+  (dimension 4.8496 (width 0.15) (layer Dwgs.User)
+    (gr_text "4.850 mm" (at 62.03 148.9548 90) (layer Dwgs.User)
+      (effects (font (size 1 1) (thickness 0.15)))
+    )
+    (feature1 (pts (xy 80.83 151.3796) (xy 62.743579 151.3796)))
+    (feature2 (pts (xy 80.83 146.53) (xy 62.743579 146.53)))
+    (crossbar (pts (xy 63.33 146.53) (xy 63.33 151.3796)))
+    (arrow1a (pts (xy 63.33 151.3796) (xy 62.743579 150.253096)))
+    (arrow1b (pts (xy 63.33 151.3796) (xy 63.916421 150.253096)))
+    (arrow2a (pts (xy 63.33 146.53) (xy 62.743579 147.656504)))
+    (arrow2b (pts (xy 63.33 146.53) (xy 63.916421 147.656504)))
+  )
+  (dimension 7.5 (width 0.15) (layer Dwgs.User)
+    (gr_text "7.500 mm" (at 77.08 154.4796) (layer Dwgs.User)
+      (effects (font (size 1 1) (thickness 0.15)))
+    )
+    (feature1 (pts (xy 80.83 151.3796) (xy 80.83 153.766021)))
+    (feature2 (pts (xy 73.33 151.3796) (xy 73.33 153.766021)))
+    (crossbar (pts (xy 73.33 153.1796) (xy 80.83 153.1796)))
+    (arrow1a (pts (xy 80.83 153.1796) (xy 79.703496 153.766021)))
+    (arrow1b (pts (xy 80.83 153.1796) (xy 79.703496 152.593179)))
+    (arrow2a (pts (xy 73.33 153.1796) (xy 74.456504 153.766021)))
+    (arrow2b (pts (xy 73.33 153.1796) (xy 74.456504 152.593179)))
+  )
   (gr_arc (start 175.6 130.8) (end 180.3 128.1) (angle -55.88761251) (layer F.SilkS) (width 0.15))
   (gr_circle (center 180.9 130.9) (end 182.5 132.5) (layer F.SilkS) (width 0.15))
@@
     (effects (font (size 2 2) (thickness 0.25)) (justify left))
   )
-  (gr_text "BrainPower Version 0.2\nhttps://github.com/Jamesits/BrainPower" (at 83 67 90) (layer B.SilkS)
+  (gr_text "BrainPower Version 0.3\nhttps://github.com/Jamesits/BrainPower" (at 194.83 138.8796) (layer B.SilkS)
     (effects (font (size 2 2) (thickness 0.25)) (justify left mirror))
   )
@@
     (arrow2b (pts (xy 241.6053 44.57192) (xy 242.191721 45.698424)))
   )
-  (dimension 7.239 (width 0.15) (layer Dwgs.User)
-    (gr_text "7.239 mm" (at 76.9493 155.8336) (layer Dwgs.User)
-      (effects (font (size 1 1) (thickness 0.15)))
-    )
-    (feature1 (pts (xy 73.3298 146.5072) (xy 73.3298 155.120021)))
-    (feature2 (pts (xy 80.5688 146.5072) (xy 80.5688 155.120021)))
-    (crossbar (pts (xy 80.5688 154.5336) (xy 73.3298 154.5336)))
-    (arrow1a (pts (xy 73.3298 154.5336) (xy 74.456304 153.947179)))
-    (arrow1b (pts (xy 73.3298 154.5336) (xy 74.456304 155.120021)))
-    (arrow2a (pts (xy 80.5688 154.5336) (xy 79.442296 153.947179)))
-    (arrow2b (pts (xy 80.5688 154.5336) (xy 79.442296 155.120021)))
-  )
-  (dimension 85.369778 (width 0.15) (layer Dwgs.User)
-    (gr_text "85.370 mm" (at 61.586891 103.765645 89.82952809) (layer Dwgs.User)
-      (effects (font (size 1 1) (thickness 0.15)))
-    )
-    (feature1 (pts (xy 80.5688 146.5072) (xy 62.173467 146.452468)))
-    (feature2 (pts (xy 80.8228 61.1378) (xy 62.427467 61.083068)))
-    (crossbar (pts (xy 63.013885 61.084813) (xy 62.759885 146.454213)))
-    (arrow1a (pts (xy 62.759885 146.454213) (xy 62.176819 145.325969)))
-    (arrow1b (pts (xy 62.759885 146.454213) (xy 63.349655 145.329459)))
-    (arrow2a (pts (xy 63.013885 61.084813) (xy 62.424115 62.209567)))
-    (arrow2b (pts (xy 63.013885 61.084813) (xy 63.596951 62.213057)))
-  )
   (gr_text ^R1 (at 205.994 85.344 90) (layer F.SilkS)
     (effects (font (size 1.5 1.5) (thickness 0.15)))
@@
     (effects (font (size 1 1) (thickness 0.15)) (justify left))
   )
-  (gr_text "BrainPower Version 0.2\nhttps://github.com/Jamesits/BrainPower" (at 83 139 90) (layer F.SilkS)
+  (gr_text "BrainPower Version 0.3\nhttps://github.com/Jamesits/BrainPower" (at 83.53 142.1296 90) (layer F.SilkS)
     (effects (font (size 2 2) (thickness 0.25)) (justify left))
   )
@@
     (effects (font (size 2 2) (thickness 0.3)))
   )
-  (gr_text 2019-10-16 (at 216.2048 193.0908) (layer Cmts.User)
+  (gr_text 2019-11-07 (at 216.2048 193.0908) (layer Cmts.User)
     (effects (font (size 2 2) (thickness 0.15)))
   )
-  (gr_text 0.2 (at 268.4272 193.0908) (layer Cmts.User)
+  (gr_text 0.3 (at 268.4272 193.0908) (layer Cmts.User)
     (effects (font (size 2 2) (thickness 0.15)) (justify left))
   )
